File: calc-matrix/calc-matrix.kicad_pcb (KiCad board)
At the start: 2 copper layers, 74 x 113 mm, 109 parts, among them J1 ESP32, J2 ESP32, J3 LiPo, J4 SD, J5 LCD, SW1 y-equals, SW10 up, SW11 stat, SW12 xton, SW13 alpha, SW14 down, SW15 left, SW16 clear, SW17 vars, SW18 prgm, SW19 red pill, SW2 window, SW20 math, SW21 carot, SW22 tan, SW23 cos, SW24 sin, SW25 x-neg1, SW26 Divide, SW27 ROFL, SW28 LOL, SW29 Comma, SW3 zoom, SW30 x-squared, SW31 Mult, SW32 9, SW33 8, SW34 7, SW35 Log, SW36 Minus, SW37 6, SW38 5, SW39 4, SW4 trace, SW40 LN, SW41 Plus, SW42 3, SW43 2, SW44 1, SW45 Sto, SW46 Enter, SW47 Neg, SW48 Dot, SW49 0, SW5 graph, SW50 PWR, SW6 del, SW7 mode, SW8 2nd, SW9 right

Commit message: v1 layout complete
Parts:
- moved J2 79.7 mm to (143.3, 133.8)
- moved J1 79.7 mm to (168.7, 133.8)
- moved D23 20.2 mm to (158.5, 81.0)
- moved D28 20.2 mm to (158.5, 91.0)
- moved D33 20.2 mm to (158.5, 101.0)
- moved D38 20.2 mm to (158.5, 111.0)
- moved D43 20.2 mm to (158.5, 121.0)
- moved D48 20.2 mm to (158.5, 131.0)
- moved D1 19.2 mm to (138.5, 31.0)
- moved D10 19.2 mm to (148.5, 40.6)
- moved D11 19.2 mm to (198.5, 61.0)
- moved D12 19.2 mm to (183.5, 61.0)
- moved D13 19.2 mm to (168.5, 61.0)
- moved D16 19.2 mm to (198.5, 71.0)
- moved D17 19.2 mm to (183.5, 71.0)
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Connections:
- J1 pad 10: COL4 -> COL7
- J1 pad 11: COL5 -> COL6
- J1 pad 12: COL6 -> COL5
- J1 pad 13: COL7 -> COL4
- J1 pad 14: COL8 -> COL3
- J1 pad 15: COL9 -> COL2
- J1 pad 16: COL10 -> COL1
- J1 pad 19: BTN_PWR -> Net-(J1-Pad19)
- J1 pad 7: COL1 -> COL10
- J1 pad 8: COL2 -> COL9
- J1 pad 9: COL3 -> COL8
- J2 pad 11: LCD_T_CLK -> LCD_BACKLIGHT
- J2 pad 12: LCD_T_CS -> LCD_SCK
- J2 pad 13: LCD_T_DIN -> LCD_MOSI
- J2 pad 14: LCD_T_DO -> LCD_DC
- J2 pad 15: LCD_T_IRQ -> LCD_RESET
- J2 pad 16: SD_CS -> LCD_CS
- J2 pad 17: SD_MOSI -> SD_CS
- J2 pad 18: SD_MISO -> SD_MOSI
- J2 pad 19: SD_SCK -> SD_MISO
- J2 pad 20: EN -> SD_SCK
- J2 pad 3: LBO -> BTN_PWR
- J2 pad 4: LCD_CS -> LBO
- J2 pad 5: LCD_RESET -> LCD_T_IRQ
- J2 pad 6: LCD_DC -> LCD_T_DO
- J2 pad 7: LCD_MOSI -> LCD_T_DIN
- J2 pad 8: LCD_SCK -> LCD_T_CS
- J2 pad 9: LCD_BACKLIGHT -> LCD_T_CLK
- J3 pad 4: EN -> +5V
Routing:
- net ROW5: track 0.00 -> 167.8 mm, vias 0 -> 3
- net ROW4: track 0.00 -> 150.7 mm, vias 0 -> 9
- net LCD_T_IRQ: track 0.00 -> 147.7 mm, vias 0 -> 2
- net LCD_T_DO: track 0.00 -> 142.0 mm, vias 0 -> 2
- net COL2: track 0.00 -> 141.2 mm, vias 0 -> 7
- net COL3: track 0.00 -> 141.2 mm, vias 0 -> 6
- net ROW1: track 0.00 -> 140.3 mm, vias 0 -> 15
- net COL1: track 0.00 -> 137.4 mm, vias 0 -> 2
- net LCD_T_DIN: track 0.00 -> 137.3 mm, vias 0 -> 2
- net LCD_T_CS: track 0.00 -> 130.1 mm, vias 0 -> 2
- net LCD_T_CLK: track 0.00 -> 125.6 mm, vias 0 -> 2
- net LCD_MISO: track 0.00 -> 121.7 mm, vias 0 -> 2
- net ROW2: track 0.00 -> 120.0 mm, vias 0 -> 10
- net LCD_BACKLIGHT: track 0.00 -> 118.5 mm, vias 0 -> 2
- net COL4: track 0.00 -> 114.7 mm, vias 0 -> 6
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
Commit message: Add some dimensions
Other:
- net class Default removed
